File: kibot.kicad_sch (KiCad schematic)
At the start: 125 parts, among them J1 ConnLeft, J2 ConnRight, SW1 SW_Push, SW10 SW_Push, SW11 SW_Push, SW12 SW_Push, SW13 SW_Push, SW14 SW_Push, SW15 SW_Push, SW16 SW_Push, SW17 SW_Push, SW18 SW_Push, SW19 SW_Push, SW2 SW_Push, SW20 SW_Push, SW21 SW_Push, SW22 SW_Push, SW23 SW_Push, SW24 SW_Push, SW25 SW_Push, SW26 SW_Push, SW27 SW_Push, SW28 SW_Push, SW29 SW_Push, SW3 SW_Push, SW30 SW_Push, SW31 SW_Push, SW32 SW_Push, SW33 SW_Push, SW34 SW_Push, SW35 SW_Push, SW36 SW_Push, SW37 SW_Push, SW38 RotaryEncoder_Switch, SW39 SW_Push, SW4 SW_Push, SW40 SW_Push, SW41 SW_Push, SW42 SW_Push, SW43 SW_Push, SW44 SW_Push, SW45 SW_Push, SW46 SW_Push, SW47 SW_Push, SW48 SW_Push, SW49 SW_Push, SW5 SW_Push, SW50 RotaryEncoder_Switch, SW51 SW_Push, SW52 SW_Push, SW53 SW_Push, SW54 SW_Push, SW55 SW_Push, SW56 SW_Push, SW57 SW_Push, SW58 SW_Push, SW59 SW_Push, SW6 SW_Push, SW60 SW_Push, SW7 SW_Push, SW8 SW_Push, SW9 SW_Push, U1 DOIT-ESP32-DEVKIT-V1

Commit message: add kicad pcb design
Parts:
- removed Oled1: ~, symbol Kibot:Oled
- removed Reset: SW_Push, symbol Switch:SW_Push
- J1, J2: footprint (none) -> Connector_IDC:IDC-Header_2x08_P2.54mm_Vertical
- SW1, SW10, SW11, SW12, SW13, SW14, SW15, SW16, SW17, SW18, SW19, SW2, SW20, SW21, SW22, SW23, SW24, SW25, SW26, SW27, SW28, SW29, SW3, SW30, SW31, SW32, SW33, SW34, SW35, SW36, SW37, SW39, SW4, SW40, SW41, SW42, SW43, SW44, SW45, SW46, SW47, SW48, SW49, SW5, SW51, SW52, SW53, SW54, SW55, SW56, SW57, SW58, SW59, SW6, SW60, SW7, SW8, SW9: footprint (none) -> Button_Switch_Keyboard:SW_Cherry_MX_1.00u_PCB
- SW38, SW50: footprint (none) -> Rotary_Encoder:RotaryEncoder_Alps_EC11E-Switch_Vertical_H20mm
Connections:
- net OledSDA is gone; now on net col11connleft: U1.32 (GPIO21_I2C-SDA)
- net Rot2EncB is gone; now on net Rot2EncAConnLeft: U1.5 (GPIO35_ADC1-CH7_RTC-GPIO5)
- net GND: no longer SW38.C, SW50.C, U1.17 (GND)
- net Rot1A: now also SW18.1, SW30.1, SW47.1, SW6.1, U1.11 (GPIO14_ADC2-CH6_HSPI-CLK_RTC-GPIO16); no longer SW1.1, SW13.1, SW25.1, SW37.1, U1.6 (GPIO32_ADC1-CH4_RTC-GPIO9)
- net Rot2A: now also J2.7 (Pin_7); no longer J2.6 (Pin_6)
- net Rot2EncA: now also J1.13 (Pin_13)
- net Rot2EncAConnLeft: now also J1.11 (Pin_11); no longer J1.12 (Pin_12), U1.34 (GPIO1_UART0-TX)
- net Rot2EncAConnRight: now also J2.5 (Pin_5); no longer J2.12 (Pin_12)
- net Rot2EncBConnRight: now also J2.3 (Pin_3); no longer J2.13 (Pin_13)
- net col1: now also SW42.1; no longer SW40.1
- net col10connleft: now also J1.4 (Pin_4); no longer J1.10 (Pin_10)
- net col10connright: now also J2.14 (Pin_14); no longer J2.10 (Pin_10)
- net col11connleft: now also J1.2 (Pin_2); no longer J1.11 (Pin_11), U1.36 (GPIO23_VSPI-MOSI)
- net col11connright: now also J2.16 (Pin_16); no longer J2.11 (Pin_11)
- net col2: now also SW44.1; no longer SW42.1
- net col3: now also SW46.1; no longer SW44.1
- net col4: now also SW48.1; no longer SW46.1
- net col6connleft: now also J1.9 (Pin_9); no longer J1.6 (Pin_6)
- net col7connright: now also J2.9 (Pin_9); no longer J2.7 (Pin_7)
- net col8connleft: now also J1.16 (Pin_16), U1.25 (GPIO2_ADC2-CH2_RTC-GPIO12); no longer J1.8 (Pin_8), U1.23 (GPIO0_ADC2-CH1_RTC-GPIO11)
- net col8connright: now also J2.2 (Pin_2); no longer J2.8 (Pin_8)
- net col9connleft: now also J1.15 (Pin_15); no longer J1.9 (Pin_9)
- net col9connright: now also J2.1 (Pin_1); no longer J2.9 (Pin_9)
- net row0: now also J1.14 (Pin_14), U1.26 (GPIO4_ADC2-CH0_RTC-GPIO10); no longer J1.1 (Pin_1), U1.30 (GPIO18_VSPI-CLK)
- net row0connright: now also J2.4 (Pin_4); no longer J2.1 (Pin_1)
- net row1: now also J1.12 (Pin_12), U1.27 (GPIO16_UART2-RX); no longer J1.2 (Pin_2), U1.29 (GPIO5_VSPI-CS0)
- net row1connright: now also J2.6 (Pin_6); no longer J2.2 (Pin_2)
- net row2: now also J1.10 (Pin_10); no longer J1.3 (Pin_3)
- net row2connright: now also J2.8 (Pin_8); no longer J2.3 (Pin_3)
- net row3: now also J1.8 (Pin_8), U1.29 (GPIO5_VSPI-CS0); no longer J1.4 (Pin_4), U1.27 (GPIO16_UART2-RX)
- net row3connright: now also J2.10 (Pin_10); no longer J2.4 (Pin_4)
- net row4: now also J1.6 (Pin_6), U1.30 (GPIO18_VSPI-CLK); no longer J1.5 (Pin_5), U1.26 (GPIO4_ADC2-CH0_RTC-GPIO10)
- net row4connright: now also J2.12 (Pin_12); no longer J2.5 (Pin_5)
- net GNDJump: now reaches J2.15 (Pin_15)
- net GNDJump: now also SW50.C
- net OledSCL: no longer names the net of U1.35 (GPIO22_I2C-SCL)
- net Rot2EncBConnLeft: no longer names the net of U1.33 (GPIO3__UART0-RX)
- net Rot2EncBConnLeft: no longer J1.13 (Pin_13)
- removed net col5: SW18.1, SW30.1, SW47.1, SW48.1, SW6.1, U1.11 (GPIO14_ADC2-CH6_HSPI-CLK_RTC-GPIO16)
- new net GndMain: J1.1 (Pin_1), SW38.C, U1.17 (GND)
- new net col0: SW1.1, SW13.1, SW25.1, SW37.1, SW40.1, U1.6 (GPIO32_ADC1-CH4_RTC-GPIO9)
- no-connect marks 6 -> 4
Other:
- note removed: "needs 6+5 = 11 pins for matrix, excluding rotary pins"
- moved on the sheet: D38, D40, D42, D44, D46, D48, SW40, SW42, SW44, SW46, SW48, U1
